Commit message: Added 1819 gripper collision mesh to urdf

File: software/ros_packages/rover_arm_urdf/urdf/rover_arm.urdf (robot description, URDF)
Before this commit: robot rover_arm, 8 links, 7 joints
Links:
- link arm_gripper: geometry collision mesh filename=package://rover_arm_urdf/urdf/stl_files/arm_1819_gripper.stl scale=0.001 0.001 0.001; visual mesh filename=package://rover_arm_urdf/urdf/dae_files/arm_gripper.dae
