Commit message: Added second depth camera configs.

File: software/ros_packages/rover_arm/config/rover_arm.urdf.xacro (robot description, xacro)
@@ -11,7 +11,12 @@
     <xacro:include filename="$(find realsense2_description)/urdf/_d405.urdf.xacro"/>
     <!-- Instantiate micros  -->
-    <xacro:sensor_d405 parent ="arm_gripper" name="camera" use_nominal_extrinsics="true">
+    <xacro:sensor_d405 parent ="arm_gripper" name="d405" use_nominal_extrinsics="true">
         <origin xyz="0 0.05 0.1" rpy="-1.5707 -1.5707 0"/>
     </xacro:sensor_d405>
+    <!-- Chassis Depth Camera -->
+    <xacro:include filename="$(find realsense2_description)/urdf/_d455.urdf.xacro"/>
+    <xacro:sensor_d455 parent="base_link" name="d455" use_nominal_extrinsics="true">
+        <origin xyz="-0.2 0.1 0" rpy="0 0 1.5707963267948"/>
+    </xacro:sensor_d455>
     <xacro:rover_arm_ros2_control name="RealSystem" initial_positions_file="$(arg initial_positions_file)" ros2_control_hardware_type="$(arg ros2_control_hardware_type)"/>
 </robot>

Commit message: Fixed controller race, octomap loading, odrive_hardware input mode

File: software/ros_packages/rover_arm/config/rover_arm.urdf.xacro (robot description, xacro)
@@ -12,5 +12,5 @@
     <!-- Instantiate micros  -->
     <xacro:sensor_d405 parent ="arm_gripper" name="d405" use_nominal_extrinsics="true">
-        <origin xyz="0 0.05 0.1" rpy="-1.5707 -1.5707 0"/>
+        <origin xyz="0 0.04075 0.1" rpy="0 -1.3963 -1.5708"/>
     </xacro:sensor_d405>
     <!-- Chassis Depth Camera -->
