Commit message: added lidar

File: description/robot.urdf.xacro (robot description, xacro)
@@ -1,5 +1,6 @@
 <?xml version="1.0"?>
-<robot xmlns:xacro="http://www.ros.org/wiki/xacro"  name="robot">
+<robot xmlns:xacro="http://www.ros.org/wiki/xacro" name="robot">
     <xacro:include filename="robot_core.xacro"/>
     <xacro:include filename="gazebo_control.xacro"/>
+    <xacro:include filename="lidar.xacro"/>
 </robot>

File: description/robot_core.xacro (robot description, xacro)
@@ -10,4 +10,7 @@
     <material name="blue">
         <color rgba="0.2 0.2 1 1"/>
+    </material>
+    <material name="red">
+        <color rgba="1 0.2 0.2 1"/>
     </material>
     <material name="black">
