Commit message: why doesnt depth slam work?

File: description/depth_camera.xacro (robot description, xacro)
@@ -57,6 +57,4 @@
         </image>
         <clip>
-          <!-- <near>0.02</near> -->
-          <!-- <far>300</far> -->
           <near>0.02</near>
           <far>300</far>
@@ -71,9 +69,13 @@
         <ros></ros>
         <!-- Topics / frame -->
-        <camera_name>camera</camera_name>
+        <camera_name>camera_depth</camera_name>
+        <frame_name>camera_rgb_optical_frame</frame_name>
+        <!-- <image_topic_name>rgb/image</image_topic_name> -->
+        <!-- <depth_image_topic_name>depth/image</depth_image_topic_name> -->
+        <!-- <camera_info_topic_name>rgb/camera_info</camera_info_topic_name> -->
+        <!-- <point_cloud_topic_name>points</point_cloud_topic_name> -->
         <image_topic_name>image_raw</image_topic_name>
         <camera_info_topic_name>camera_info</camera_info_topic_name>
         <point_cloud_topic_name>points</point_cloud_topic_name>
-        <frame_name>camera_rgb_optical_frame</frame_name>
         <!-- useful plugin params you can tune -->
         <update_rate>30</update_rate>
@@ -81,5 +83,5 @@
         <visualize>true</visualize>
         <min_depth>0.02</min_depth>
-        <max_depth>200</max_depth>
+        <max_depth>50.0</max_depth>
       </plugin>
     </sensor>

File: description/robot_core.xacro (robot description, xacro)
@@ -20,4 +20,5 @@
     <link name="base_link" />
     <!-- BASE FOOTPRINT LINK-->
+    <link name="base_footprint" />
     <joint name="base_footprint_joint" type="fixed">
         <parent link="base_link"/>
@@ -25,5 +26,4 @@
         <origin xyz="0 0 0" rpy="0 0 0"/>
     </joint>
-    <link name="base_footprint" />
     <!-- CHASSIS LINK -->
     <joint name="chassis_joint" type="fixed">
